Commit message: add apply force

File: resources/robots/go1/urdf/go1_v2.urdf (robot description, URDF)
Before this commit: robot go1_description, 23 links, 22 joints
Links:
- link FL_calf: mass 0.135862 -> 0.158015
- link FL_hip: mass 0.68 -> 0.510299
- link FL_thigh: mass 0.92 -> 0.898919
- link FR_calf: mass 0.135862 -> 0.158015
- link FR_hip: mass 0.68 -> 0.510299
- link FR_thigh: mass 0.92 -> 0.898919
- link RL_calf: mass 0.135862 -> 0.158015
- link RL_hip: mass 0.68 -> 0.510299
- link RL_thigh: mass 0.92 -> 0.898919
- link RR_calf: mass 0.135862 -> 0.158015
- link RR_hip: mass 0.68 -> 0.510299
- link RR_thigh: mass 0.92 -> 0.898919
- link trunk: mass 5.916 -> 6.49
Joints:
- joint FL_calf_joint: limit lower=-2.69653369433 upper=-0.916297857297 effort=33.5 velocity=28 -> lower=-2.818 upper=-0.888 effort=35.55 velocity=20.06
- joint FL_hip_joint: limit lower=-0.802851455917 upper=0.802851455917 effort=33.5 velocity=50 -> lower=-0.863 upper=0.863 effort=23.7 velocity=30.1
- joint FL_thigh_joint: limit lower=-1.0471975512 upper=4.18879020479 effort=33.5 velocity=28 -> lower=-0.686 upper=4.501 effort=23.7 velocity=30.1
- joint FR_calf_joint: limit lower=-2.69653369433 upper=-0.916297857297 effort=33.5 velocity=28 -> lower=-2.818 upper=-0.888 effort=35.55 velocity=20.06
- joint FR_hip_joint: limit lower=-0.802851455917 upper=0.802851455917 effort=33.5 velocity=50 -> lower=-0.863 upper=0.863 effort=23.7 velocity=30.1
- joint FR_thigh_joint: limit lower=-1.0471975512 upper=4.18879020479 effort=33.5 velocity=28 -> lower=-0.686 upper=4.501 effort=23.7 velocity=30.1
- joint RL_calf_joint: limit lower=-2.69653369433 upper=-0.916297857297 effort=33.5 velocity=28 -> lower=-2.818 upper=-0.888 effort=35.55 velocity=20.06
- joint RL_hip_joint: limit lower=-0.802851455917 upper=0.802851455917 effort=33.5 velocity=50 -> lower=-0.863 upper=0.863 effort=23.7 velocity=30.1
- joint RL_thigh_joint: limit lower=-1.0471975512 upper=4.18879020479 effort=33.5 velocity=28 -> lower=-0.686 upper=4.501 effort=23.7 velocity=30.1
- joint RR_calf_joint: limit lower=-2.69653369433 upper=-0.916297857297 effort=33.5 velocity=28 -> lower=-2.818 upper=-0.888 effort=35.55 velocity=20.06
- joint RR_hip_joint: limit lower=-0.802851455917 upper=0.802851455917 effort=33.5 velocity=50 -> lower=-0.863 upper=0.863 effort=23.7 velocity=30.1
- joint RR_thigh_joint: limit lower=-1.0471975512 upper=4.18879020479 effort=33.5 velocity=28 -> lower=-0.686 upper=4.501 effort=23.7 velocity=30.1
